Commit message: updates

File: example/bin/data/relaxed_ik_core/config/urdfs/irb120.urdf (robot description, URDF)
Before this commit: robot abb_irb120, 9 links, 8 joints
Links:
- link base_link: geometry collision mesh filename=meshes/irb120/collision/base_link.stl; visual mesh filename=meshes/irb120/visual/base_link.stl
- link link_1: geometry collision mesh filename=meshes/irb120/collision/link_1.stl; visual mesh filename=meshes/irb120/visual/link_1.stl
- link link_2: geometry collision mesh filename=meshes/irb120/collision/link_2.stl; visual mesh filename=meshes/irb120/visual/link_2.stl
- link link_3: geometry collision mesh filename=meshes/irb120/collision/link_3.stl; visual mesh filename=meshes/irb120/visual/link_3.stl
- link link_4: geometry collision mesh filename=meshes/irb120/collision/link_4.stl; visual mesh filename=meshes/irb120/visual/link_4.stl
- link link_5: geometry collision mesh filename=meshes/irb120/collision/link_5.stl; visual mesh filename=meshes/irb120/visual/link_5.stl
- link link_6: geometry collision mesh filename=meshes/irb120/collision/link_6.stl; visual mesh filename=meshes/irb120/visual/link_6.stl
