Commit message: adding xarm

File: example-urdf/bin/data/relaxed_ik_core/config/urdfs/irb120.urdf (robot description, URDF)
Before this commit: robot abb_irb120, 9 links, 8 joints
Links:
- link base_link: geometry collision mesh filename=package://abb_irb120_support/meshes/irb120/collision/base_l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; visual mesh filename=package://abb_irb120_support/meshes/irb120/visual/base_link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
- link link_1: geometry collision mesh filename=package://abb_irb120_support/meshes/irb120/collision/link_1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; visual mesh filename=package://abb_irb120_support/meshes/irb120/visual/link_1.stl
- link link_2: geometry collision mesh filename=package://abb_irb120_support/meshes/irb120/collision/link_2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; visual mesh filename=package://abb_irb120_support/meshes/irb120/visual/link_2.stl
- link link_3: geometry collision mesh filename=package://abb_irb120_support/meshes/irb120/collision/link_3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; visual mesh filename=package://abb_irb120_support/meshes/irb120/visual/link_3.stl
- link link_4: geometry collision mesh filename=package://abb_irb120_support/meshes/irb120/collision/link_4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; visual mesh filename=package://abb_irb120_support/meshes/irb120/visual/link_4.stl
- link link_5: geometry collision mesh filename=package://abb_irb120_support/meshes/irb120/collision/link_5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; visual mesh filename=package://abb_irb120_support/meshes/irb120/visual/link_5.stl
- link link_6: geometry collision mesh filename=package://abb_irb120_support/meshes/irb120/collision/link_6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; visual mesh filename=package://abb_irb120_support/meshes/irb120/visual/link_6.stl

File: example-urdf/bin/data/relaxed_ik_core/config/urdfs/ur10.urdf (robot description, URDF)
Before this commit: robot ur10, 11 links, 10 joints
Links:
- link base_link: geometry collision mesh filename=package://ur_description/meshes/ur10/collision/base.stl; visual mesh filename=package://ur_description/meshes/ur10/visual/base.dae
- link forearm_link: geometry collision mesh filename=package://ur_description/meshes/ur10/collision/forearm.stl; visual mesh filename=package://ur_description/meshes/ur10/visual/forearm.dae
- link shoulder_link: geometry collision mesh filename=package://ur_description/meshes/ur10/collision/shoulder.stl; visual mesh filename=package://ur_description/meshes/ur10/visual/shoulder.dae
- link upper_arm_link: geometry collision mesh filename=package://ur_description/meshes/ur10/collision/upperarm.stl; visual mesh filename=package://ur_description/meshes/ur10/visual/upperarm.dae
- link wrist_1_link: geometry collision mesh filename=package://ur_description/meshes/ur10/collision/wrist1.stl; visual mesh filename=package://ur_description/meshes/ur10/visual/wrist1.dae
- link wrist_2_link: geometry collision mesh filename=package://ur_description/meshes/ur10/collision/wrist2.stl; visual mesh filename=package://ur_description/meshes/ur10/visual/wrist2.dae
- link wrist_3_link: geometry collision mesh filename=package://ur_description/meshes/ur10/collision/wrist3.stl; visual mesh filename=package://ur_description/meshes/ur10/visual/wrist3.dae

File: example-urdf/bin/data/relaxed_ik_core/config/urdfs/ur5.urdf (robot description, URDF)
Before this commit: robot ur5, 9 links, 8 joints
Links:
- added link base
- added link tool0
- link base_link: geometry collision mesh filename=package://ur_description/meshes/ur5/collision/base.stl; visual mesh filename=package://ur_description/meshes/ur5/visual/base.dae
- link forearm_link: geometry collision mesh filename=package://ur_description/meshes/ur5/collision/forearm.stl; visual mesh filename=package://ur_description/meshes/ur5/visual/forearm.dae
- link shoulder_link: geometry collision mesh filename=package://ur_description/meshes/ur5/collision/shoulder.stl; visual mesh filename=package://ur_description/meshes/ur5/visual/shoulder.dae
- link upper_arm_link: geometry collision mesh filename=package://ur_description/meshes/ur5/collision/upperarm.stl; visual mesh filename=package://ur_description/meshes/ur5/visual/upperarm.dae
- link wrist_1_link: geometry collision mesh filename=package://ur_description/meshes/ur5/collision/wrist1.stl; visual mesh filename=package://ur_description/meshes/ur5/visual/wrist1.dae
- link wrist_2_link: geometry collision mesh filename=package://ur_description/meshes/ur5/collision/wrist2.stl; visual mesh filename=package://ur_description/meshes/ur5/visual/wrist2.dae
- link wrist_3_link: geometry collision mesh filename=package://ur_description/meshes/ur5/collision/wrist3.stl; visual mesh filename=package://ur_description/meshes/ur5/visual/wrist3.dae
Joints:
- added joint base_link-base_fixed_joint: type fixed, parent base_link, child base, origin xyz=0 0 0 rpy=0 0 -3.14159265
- added joint wrist_3_link-tool0_fixed_joint: type fixed, parent wrist_3_link, child tool0, origin xyz=0 0.0823 0 rpy=-1.570796325 0 0
- joint shoulder_lift_joint: origin xyz=0.0 0.13585 0.0 rpy=0.0 1.570796325 0.0 -> xyz=0.0 0.13585 0.0 rpy=0.0 0.0 0.0
- joint wrist_1_joint: origin xyz=0.0 0.0 0.39225 rpy=0.0 1.570796325 0.0 -> xyz=0.0 0.0 0.39225 rpy=0.0 0.0 0.0
