Commit message: updates

File: example-urdf/bin/data/relaxed_ik_core/config/urdfs/ur10.urdf (robot description, URDF)
Before this commit: robot ur10, 11 links, 10 joints
Links:
- link base_link: geometry collision mesh filename=meshes/ur10/collision/base.stl; visual mesh filename=meshes/ur10/visual/base.dae
- link forearm_link: geometry collision mesh filename=meshes/ur10/collision/forearm.stl; visual mesh filename=meshes/ur10/visual/forearm.dae
- link shoulder_link: geometry collision mesh filename=meshes/ur10/collision/shoulder.stl; visual mesh filename=meshes/ur10/visual/shoulder.dae
- link upper_arm_link: geometry collision mesh filename=meshes/ur10/collision/upperarm.stl; visual mesh filename=meshes/ur10/visual/upperarm.dae
- link wrist_1_link: geometry collision mesh filename=meshes/ur10/collision/wrist1.stl; visual mesh filename=meshes/ur10/visual/wrist1.dae
- link wrist_2_link: geometry collision mesh filename=meshes/ur10/collision/wrist2.stl; visual mesh filename=meshes/ur10/visual/wrist2.dae
- link wrist_3_link: geometry collision mesh filename=meshes/ur10/collision/wrist3.stl; visual mesh filename=meshes/ur10/visual/wrist3.dae
