Commit message: updates

File: example-urdf/bin/data/relaxed_ik_core/config/urdfs/ur5.urdf (robot description, URDF)
Before this commit: robot ur5, 9 links, 8 joints
Links:
- link base_link: geometry collision mesh filename=meshes/ur5/collision/base.stl; visual mesh filename=meshes/ur5/visual/base.dae
- link forearm_link: geometry collision mesh filename=meshes/ur5/collision/forearm.stl; visual mesh filename=meshes/ur5/visual/forearm.dae
- link shoulder_link: geometry collision mesh filename=meshes/ur5/collision/shoulder.stl; visual mesh filename=meshes/ur5/visual/shoulder.dae
- link upper_arm_link: geometry collision mesh filename=meshes/ur5/collision/upper_arm.stl; visual mesh filename=meshes/ur5/visual/upperarm.dae
- link wrist_1_link: geometry collision mesh filename=meshes/ur5/collision/wrist_1.stl; visual mesh filename=meshes/ur5/visual/wrist1.dae
- link wrist_2_link: geometry collision mesh filename=meshes/ur5/collision/wrist_2.stl; visual mesh filename=meshes/ur5/visual/wrist2.dae
- link wrist_3_link: geometry collision mesh filename=meshes/ur5/collision/wrist_3.stl; visual mesh filename=meshes/ur5/visual/wrist3.dae

Commit message: correct UR5 urdf for the trained network

File: example-urdf/bin/data/relaxed_ik_core/config/urdfs/ur5.urdf (robot description, URDF)
Before this commit: robot ur5, 11 links, 10 joints
Joints:
- joint base_link-base_fixed_joint: origin xyz=0 0 0 rpy=0 0 -3.14159265 -> xyz=0 0 0 rpy=0 0 -3.14159265359
- joint ee_fixed_joint: origin xyz=0.0 0.0823 0.0 rpy=0.0 0.0 1.570796325 -> xyz=0.0 0.0823 0.0 rpy=0.0 0.0 1.57079632679
- joint elbow_joint: limit lower=-6.2831853 upper=6.2831853 effort=150.0 velocity=3.15 -> lower=-3.14159265359 upper=3.14159265359 effort=150.0 velocity=3.15
- joint shoulder_lift_joint: limit lower=-6.2831853 upper=6.2831853 effort=150.0 velocity=3.15 -> lower=-6.28318530718 upper=6.28318530718 effort=150.0 velocity=3.15; origin xyz=0.0 0.13585 0.0 rpy=0.0 0.0 0.0 -> xyz=0.0 0.13585 0.0 rpy=0.0 1.57079632679 0.0
- joint shoulder_pan_joint: limit lower=-6.2831853 upper=6.2831853 effort=150.0 velocity=3.15 -> lower=-6.28318530718 upper=6.28318530718 effort=150.0 velocity=3.15
- joint wrist_1_joint: limit lower=-6.2831853 upper=6.2831853 effort=28.0 velocity=3.2 -> lower=-6.28318530718 upper=6.28318530718 effort=28.0 velocity=3.2; origin xyz=0.0 0.0 0.39225 rpy=0.0 0.0 0.0 -> xyz=0.0 0.0 0.39225 rpy=0.0 1.57079632679 0.0
- joint wrist_2_joint: limit lower=-6.2831853 upper=6.2831853 effort=28.0 velocity=3.2 -> lower=-6.28318530718 upper=6.28318530718 effort=28.0 velocity=3.2
- joint wrist_3_joint: limit lower=-6.2831853 upper=6.2831853 effort=28.0 velocity=3.2 -> lower=-6.28318530718 upper=6.28318530718 effort=28.0 velocity=3.2
- joint wrist_3_link-tool0_fixed_joint: origin xyz=0 0.0823 0 rpy=-1.570796325 0 0 -> xyz=0 0.0823 0 rpy=-1.57079632679 0 0
