Commit message: tweaks

File: example-urdf/bin/data/relaxed_ik_core/config/urdfs/panda_arm_hand.urdf (robot description, URDF)
Before this commit: robot panda, 13 links, 12 joints
Links:
- link panda_hand: geometry collision mesh filename=meshes/panda/collision/hand.stl; visual mesh filename=meshes/panda/visual/hand.dae
- link panda_leftfinger: geometry collision mesh filename=meshes/panda/collision/finger.stl; visual mesh filename=meshes/panda/visual/finger.dae
- link panda_link0: geometry collision mesh filename=meshes/panda/collision/link0.stl; visual mesh filename=meshes/panda/visual/link0.dae
- link panda_link1: geometry collision mesh filename=meshes/panda/collision/link1.stl; visual mesh filename=meshes/panda/visual/link1.dae
- link panda_link2: geometry collision mesh filename=meshes/panda/collision/link2.stl; visual mesh filename=meshes/panda/visual/link2.dae
- link panda_link3: geometry collision mesh filename=meshes/panda/collision/link3.stl; visual mesh filename=meshes/panda/visual/link3.dae
- link panda_link4: geometry collision mesh filename=meshes/panda/collision/link4.stl; visual mesh filename=meshes/panda/visual/link4.dae
- link panda_link5: geometry collision mesh filename=meshes/panda/collision/link5.stl; visual mesh filename=meshes/panda/visual/link5.dae
- link panda_link6: geometry collision mesh filename=meshes/panda/collision/link6.stl; visual mesh filename=meshes/panda/visual/link6.dae
- link panda_link7: geometry collision mesh filename=meshes/panda/collision/link7.stl; visual mesh filename=meshes/panda/visual/link7.dae
- link panda_rightfinger: geometry collision mesh filename=meshes/panda/collision/finger.stl; visual mesh filename=meshes/panda/visual/finger.dae

Commit message: adding 4600

File: example-urdf/bin/data/relaxed_ik_core/config/urdfs/panda_arm_hand.urdf (robot description, URDF)
Before this commit: robot panda, 13 links, 12 joints
Links:
- link panda_hand: geometry collision mesh filename=package://franka_gazebo/meshes/collision/hand.stl; visual mesh filename=package://franka_gazebo/meshes/visual/hand.dae
- link panda_leftfinger: geometry collision mesh filename=package://franka_gazebo/meshes/collision/finger.stl; visual mesh filename=package://franka_gazebo/meshes/visual/finger.dae
- link panda_link0: geometry collision mesh filename=package://franka_gazebo/meshes/collision/link0.stl; visual mesh filename=package://franka_gazebo/meshes/visual/link0.dae
- link panda_link1: geometry collision mesh filename=package://franka_gazebo/meshes/collision/link1.stl; visual mesh filename=package://franka_gazebo/meshes/visual/link1.dae
- link panda_link2: geometry collision mesh filename=package://franka_gazebo/meshes/collision/link2.stl; visual mesh filename=package://franka_gazebo/meshes/visual/link2.dae
- link panda_link3: geometry collision mesh filename=package://franka_gazebo/meshes/collision/link3.stl; visual mesh filename=package://franka_gazebo/meshes/visual/link3.dae
- link panda_link4: geometry collision mesh filename=package://franka_gazebo/meshes/collision/link4.stl; visual mesh filename=package://franka_gazebo/meshes/visual/link4.dae
- link panda_link5: geometry collision mesh filename=package://franka_gazebo/meshes/collision/link5.stl; visual mesh filename=package://franka_gazebo/meshes/visual/link5.dae
- link panda_link6: geometry collision mesh filename=package://franka_gazebo/meshes/collision/link6.stl; visual mesh filename=package://franka_gazebo/meshes/visual/link6.dae
- link panda_link7: geometry collision mesh filename=package://franka_gazebo/meshes/collision/link7.stl; visual mesh filename=package://franka_gazebo/meshes/visual/link7.dae
- link panda_rightfinger: geometry collision mesh filename=package://franka_gazebo/meshes/collision/finger.stl; visual mesh filename=package://franka_gazebo/meshes/visual/finger.dae

File: example-urdf/bin/data/relaxed_ik_core/config/urdfs/ur5.urdf (robot description, URDF)
Before this commit: robot ur5, 11 links, 10 joints
Links:
- link base_link: geometry collision mesh filename=package://ur_description/meshes/ur5/collision/base.stl; visual mesh filename=package://ur_description/meshes/ur5/visual/base.dae
- link forearm_link: geometry collision mesh filename=package://ur_description/meshes/ur5/collision/forearm.stl; visual mesh filename=package://ur_description/meshes/ur5/visual/forearm.dae
- link shoulder_link: geometry collision mesh filename=package://ur_description/meshes/ur5/collision/shoulder.stl; visual mesh filename=package://ur_description/meshes/ur5/visual/shoulder.dae
- link upper_arm_link: geometry collision mesh filename=package://ur_description/meshes/ur5/collision/upperarm.stl; visual mesh filename=package://ur_description/meshes/ur5/visual/upperarm.dae
- link wrist_1_link: geometry collision mesh filename=package://ur_description/meshes/ur5/collision/wrist1.stl; visual mesh filename=package://ur_description/meshes/ur5/visual/wrist1.dae
- link wrist_2_link: geometry collision mesh filename=package://ur_description/meshes/ur5/collision/wrist2.stl; visual mesh filename=package://ur_description/meshes/ur5/visual/wrist2.dae
- link wrist_3_link: geometry collision mesh filename=package://ur_description/meshes/ur5/collision/wrist3.stl; visual mesh filename=package://ur_description/meshes/ur5/visual/wrist3.dae
Joints:
- joint base_link-base_fixed_joint: origin xyz=0 0 0 rpy=0 0 -3.14159265359 -> xyz=0 0 0 rpy=0 0 -3.14159265
- joint ee_fixed_joint: origin xyz=0.0 0.0823 0.0 rpy=0.0 0.0 1.57079632679 -> xyz=0.0 0.0823 0.0 rpy=0.0 0.0 1.570796325
- joint elbow_joint: limit lower=-3.14159265359 upper=3.14159265359 effort=150.0 velocity=3.15 -> lower=-6.2831853 upper=6.2831853 effort=150.0 velocity=3.15
- joint shoulder_lift_joint: limit lower=-6.28318530718 upper=6.28318530718 effort=150.0 velocity=3.15 -> lower=-6.2831853 upper=6.2831853 effort=150.0 velocity=3.15; origin xyz=0.0 0.13585 0.0 rpy=0.0 1.57079632679 0.0 -> xyz=0.0 0.13585 0.0 rpy=0.0 0.0 0.0
- joint shoulder_pan_joint: limit lower=-6.28318530718 upper=6.28318530718 effort=150.0 velocity=3.15 -> lower=-6.2831853 upper=6.2831853 effort=150.0 velocity=3.15
- joint wrist_1_joint: limit lower=-6.28318530718 upper=6.28318530718 effort=28.0 velocity=3.2 -> lower=-6.2831853 upper=6.2831853 effort=28.0 velocity=3.2; origin xyz=0.0 0.0 0.39225 rpy=0.0 1.57079632679 0.0 -> xyz=0.0 0.0 0.39225 rpy=0.0 0.0 0.0
- joint wrist_2_joint: limit lower=-6.28318530718 upper=6.28318530718 effort=28.0 velocity=3.2 -> lower=-6.2831853 upper=6.2831853 effort=28.0 velocity=3.2
- joint wrist_3_joint: limit lower=-6.28318530718 upper=6.28318530718 effort=28.0 velocity=3.2 -> lower=-6.2831853 upper=6.2831853 effort=28.0 velocity=3.2
- joint wrist_3_link-tool0_fixed_joint: origin xyz=0 0.0823 0 rpy=-1.57079632679 0 0 -> xyz=0 0.0823 0 rpy=-1.570796325 0 0
